File: kicad_6_docs/phase_inverter.kicad_sch (KiCad schematic)
At the start: 14 parts

Commit message: fix  component val, tidy up
Other:
- moved on the sheet: R19
Changed lines of the file:
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@@
   (junction (at 147.32 72.39) (diameter 0) (color 0 0 0 0)
   )
-  (junction (at 195.58 40.64) (diameter 0) (color 0 0 0 0)
-  )
   (junction (at 105.41 88.9) (diameter 0) (color 0 0 0 0)
   )
+  (junction (at 195.58 48.26) (diameter 0) (color 0 0 0 0)
+  )
   (junction (at 114.3 88.9) (diameter 0) (color 0 0 0 0)
   )
@@
   (junction (at 92.71 88.9) (diameter 0) (color 0 0 0 0)
   )
-  (junction (at 144.78 142.24) (diameter 0) (color 0 0 0 0)
-  )
-  (junction (at 168.91 142.24) (diameter 0) (color 0 0 0 0)
+  (junction (at 144.78 123.19) (diameter 0) (color 0 0 0 0)
+  )
+  (junction (at 168.91 123.19) (diameter 0) (color 0 0 0 0)
   )
   (wire (pts (xy 187.96 88.9) (xy 180.34 88.9))
@@
     (stroke (width 0) (type default) (color 0 0 0 0))
   )
-  (wire (pts (xy 193.04 142.24) (xy 193.04 120.65))
-    (stroke (width 0) (type default) (color 0 0 0 0))
-  )
-  (wire (pts (xy 85.09 104.14) (xy 85.09 142.24))
+  (wire (pts (xy 193.04 123.19) (xy 193.04 120.65))
+    (stroke (width 0) (type default) (color 0 0 0 0))
+  )
+  (wire (pts (xy 85.09 120.65) (xy 85.09 123.19))
     (stroke (width 0) (type default) (color 0 0 0 0))
   )
@@
     (stroke (width 0) (type default) (color 0 0 0 0))
   )
-  (wire (pts (xy 144.78 120.65) (xy 144.78 142.24))
+  (wire (pts (xy 144.78 120.65) (xy 144.78 123.19))
     (stroke (width 0) (type default) (color 0 0 0 0))
   )
@@
     (stroke (width 0) (type default) (color 0 0 0 0))
   )
-  (wire (pts (xy 168.91 142.24) (xy 168.91 148.59))
+  (wire (pts (xy 168.91 123.19) (xy 168.91 125.73))
     (stroke (width 0) (type default) (color 0 0 0 0))
   )
@@
     (stroke (width 0) (type default) (color 0 0 0 0))
   )
-  (wire (pts (xy 195.58 58.42) (xy 195.58 40.64))
+  (wire (pts (xy 195.58 58.42) (xy 195.58 48.26))
     (stroke (width 0) (type default) (color 0 0 0 0))
   )
@@
     (stroke (width 0) (type default) (color 0 0 0 0))
   )
-  (wire (pts (xy 147.32 59.69) (xy 147.32 40.64))
+  (wire (pts (xy 147.32 59.69) (xy 147.32 48.26))
     (stroke (width 0) (type default) (color 0 0 0 0))
   )
@@
     (stroke (width 0) (type default) (color 0 0 0 0))
   )
-  (wire (pts (xy 147.32 40.64) (xy 195.58 40.64))
+  (wire (pts (xy 147.32 48.26) (xy 195.58 48.26))
     (stroke (width 0) (type default) (color 0 0 0 0))
   )
@@
     (stroke (width 0) (type default) (color 0 0 0 0))
   )
-  (wire (pts (xy 85.09 142.24) (xy 144.78 142.24))
+  (wire (pts (xy 85.09 123.19) (xy 144.78 123.19))
     (stroke (width 0) (type default) (color 0 0 0 0))
   )
@@
     (stroke (width 0) (type default) (color 0 0 0 0))
   )
-  (wire (pts (xy 144.78 142.24) (xy 168.91 142.24))
+  (wire (pts (xy 144.78 123.19) (xy 168.91 123.19))
     (stroke (width 0) (type default) (color 0 0 0 0))
   )
@@
     (stroke (width 0) (type default) (color 0 0 0 0))
   )
-  (wire (pts (xy 203.2 40.64) (xy 195.58 40.64))
-    (stroke (width 0) (type default) (color 0 0 0 0))
-  )
-  (wire (pts (xy 85.09 96.52) (xy 85.09 88.9))
-    (stroke (width 0) (type default) (color 0 0 0 0))
-  )
-  (wire (pts (xy 168.91 142.24) (xy 193.04 142.24))
-    (stroke (width 0) (type default) (color 0 0 0 0))
-  )
-  (global_label "B+_3" (shape input) (at 203.2 40.64 0) (fields_autoplaced)
+  (wire (pts (xy 203.2 48.26) (xy 195.58 48.26))
+    (stroke (width 0) (type default) (color 0 0 0 0))
+  )
+  (wire (pts (xy 85.09 113.03) (xy 85.09 88.9))
+    (stroke (width 0) (type default) (color 0 0 0 0))
+  )
+  (wire (pts (xy 168.91 123.19) (xy 193.04 123.19))
+    (stroke (width 0) (type default) (color 0 0 0 0))
+  )
+  (global_label "B+_3" (shape input) (at 203.2 48.26 0) (fields_autoplaced)
     (effects (font (size 1.27 1.27)) (justify left))
-    (property "Intersheet References" "${INTERSHEET_REFS}" (id 0) (at 30.48 -2.54 0)
+    (property "Intersheet References" "${INTERSHEET_REFS}" (id 0) (at 30.48 5.08 0)
       (effects (font (size 1.27 1.27)) hide)
     )
@@
     (pin "2")
   )
-  (symbol (lib_id "power:GND") (at 168.91 148.59 0) (unit 1)
-    (in_bom yes) (on_board yes)
-    (property "Reference" "#PWR08" (id 0) (at 168.91 154.94 0)
-      (effects (font (size 1.27 1.27)) hide)
-    )
-    (property "Value" "GND" (id 1) (at 169.037 152.9842 0))
-    (property "Footprint" "" (id 2) (at 168.91 148.59 0)
-      (effects (font (size 1.27 1.27)) hide)
-    )
-    (property "Datasheet" "" (id 3) (at 168.91 148.59 0)
+  (symbol (lib_id "power:GND") (at 168.91 125.73 0) (unit 1)
+    (in_bom yes) (on_board yes)
+    (property "Reference" "#PWR08" (id 0) (at 168.91 132.08 0)
+      (effects (font (size 1.27 1.27)) hide)
+    )
+    (property "Value" "GND" (id 1) (at 169.037 130.1242 0))
+    (property "Footprint" "" (id 2) (at 168.91 125.73 0)
+      (effects (font (size 1.27 1.27)) hide)
+    )
+    (property "Datasheet" "" (id 3) (at 168.91 125.73 0)
       (effects (font (size 1.27 1.27)) hide)
     )
@@
     (pin "2")
   )
-  (symbol (lib_id "Device:R_Photo") (at 85.09 100.33 0) (mirror x) (unit 1)
+  (symbol (lib_id "Device:R_Photo") (at 85.09 116.84 0) (mirror x) (unit 1)
     (in_bom yes) (on_board yes) (fields_autoplaced)
-    (property "Reference" "R19" (id 0) (at 80.01 99.0599 0)
+    (property "Reference" "R19" (id 0) (at 80.01 115.5699 0)
       (effects (font (size 1.27 1.27)) (justify right))
     )
-    (property "Value" "trem_opto" (id 1) (at 80.01 101.5999 0)
+    (property "Value" "trem_opto" (id 1) (at 80.01 118.1099 0)
       (effects (font (size 1.27 1.27)) (justify right))
     )
-    (property "Footprint" "" (id 2) (at 86.36 93.98 90)
+    (property "Footprint" "" (id 2) (at 86.36 110.49 90)
       (effects (font (size 1.27 1.27)) (justify left) hide)
     )
-    (property "Datasheet" "~" (id 3) (at 85.09 99.06 0)
-      (effects (font (size 1.27 1.27)) hide)
-    )
+    (property "Datasheet" "~" (id 3) (at 85.09 115.57 0)
+      (effects (font (size 1.27 1.27)) hide)
+    )
