File: kicad_6_docs/preamp.kicad_sch (KiCad schematic)
At the start: 25 parts

Commit message: fix  component val, tidy up
Parts:
- C7: value 4n7 450v -> 100n
Changed lines of the file:
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@@
     (in_bom yes) (on_board yes)
     (property "Reference" "C7" (id 0) (at 241.3 101.5492 90))
-    (property "Value" "4n7 450v" (id 1) (at 241.3 103.8606 90))
+    (property "Value" "100n" (id 1) (at 241.3 103.8606 90))
     (property "Footprint" "" (id 2) (at 237.49 108.9152 0)
       (effects (font (size 1.27 1.27)) hide)
